Commit message: transform added

File: src/reachy_vel_description/urdf/reachy.urdf (robot description, URDF)
Before this commit: robot Reachy, 10 links, 9 joints
Links:
- link kinect: geometry collision mesh filename=package://reachy_vel_description/meshes/kinect.dae; visual mesh filename=package://reachy_vel_description/meshes/kinect.dae

Commit message: wrist roll removed

File: src/reachy_vel_description/urdf/reachy.urdf (robot description, URDF)
Before this commit: robot Reachy, 10 links, 9 joints
Joints:
- joint wrist_roll: axis 1 0 0 -> (none); origin xyz=0 0 -0.03243 rpy=0 0 0 -> (none); type revolute -> fixed

Commit message: hand_ball removed

File: src/reachy_vel_description/urdf/reachy.urdf (robot description, URDF)
Before this commit: robot Reachy, 10 links, 9 joints
Links:
- removed link hand_ball
Joints:
- removed joint wrist_roll
- joint kinect_hand: parent hand_ball -> wrist_hand

Commit message: Kacobian updated

File: src/reachy_vel_description/urdf/reachy.urdf (robot description, URDF)
Before this commit: robot Reachy, 10 links, 9 joints
Links:
- removed link hand_ball
- link kinect: geometry collision mesh filename=package://reachy_vel_description/meshes/kinect.dae; visual mesh filename=package://reachy_vel_description/meshes/kinect.dae
Joints:
- removed joint wrist_roll
- joint kinect_hand: parent hand_ball -> wrist_hand

Commit message: init added

File: src/reachy_vel_description/urdf/reachy.urdf (robot description, URDF)
Before this commit: robot Reachy, 9 links, 8 joints
Joints:
- joint kinect_hand: axis (none) -> 0.0 1.0 0.0

Commit message: Depth calculation using RGB

File: src/reachy_vel_description/urdf/reachy.urdf (robot description, URDF)
Before this commit: robot Reachy, 9 links, 8 joints
Joints:
- joint kinect_hand: limit lower=3.0 upper=3.0 effort=3.0 velocity=0.0 -> lower=0.0 upper=0.0 effort=0.0 velocity=0.0; type fixed -> revolute
